File: motorControllerMk3/motorControllerMk3.sch (EAGLE design)
At the start: 28 parts, among them IC1 VNH3SP30, IC2 VNH3SP30

Commit message: developing schematics
Parts:
- added C8: 2200u, rcl:CPOL-EUE5-8.5
- added LED5, LED6: (no value), led:LEDSML1206
- added R10, R12, R13, R14, R15, R16, R17: 1k, rcl:R-EU_M0805
- added R11: 3k3, rcl:R-EU_M0805
- C1, C2: value (none) -> 22p
- C3: value (none) -> 1n
- C4, C5, C6, C7: value (none) -> 100n
- R2, R3, R4, R5: value (none) -> 3k3
- R6, R7, R8, R9: value (none) -> 1k
Connections:
- new net N$28: LED5.A, R10.1
- new net N$29: LED6.A, R11.1
- new net N$32: IC1.INA, R12.1
- new net N$33: IC1.INB, R13.1
- new net N$34: IC1.PWM, R14.1
- new net N$35: IC2.INA, R15.1
- new net N$36: IC2.PWM, R17.1
- new net N$37: IC2.INB, R16.1
- net +12V: now also C8.+, R11.2
- net +5V: now also R10.2
- net GND: now also C8.-, LED5.C, LED6.C
- net N$23: now also R16.2; no longer IC2.INB
- net N$24: now also R15.2; no longer IC2.INA
- net N$25: now also R13.2; no longer IC1.INB
- net N$26: now also R12.2; no longer IC1.INA
- net N$8: now also R17.2; no longer IC2.PWM
- net N$9: now also R14.2; no longer IC1.PWM
Other:
- moved on the sheet: IC1, IC2, SV1, SV2

Commit message: finished layout
Connections:
- net N$15: now also SV2.6; no longer SV2.5
- net N$16: now also SV2.5; no longer SV2.6
- net N$24: now also R12.2, U$1.PB4(ADC11); no longer R15.2, U$1.PD5(XCK/CTS)
- net N$25: now also R15.2; no longer R13.2
- net N$26: now also R13.2; no longer R12.2
Changed lines of the file:
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@@
 <?xml version="1.0" encoding="utf-8"?>
 <!DOCTYPE eagle SYSTEM "eagle.dtd">
-<eagle version="6.3">
+<eagle version="6.5.0">
 <drawing>
 <settings>
@@
 <wire x1="129.54" y1="20.32" x2="129.54" y2="22.86" width="0.1524" layer="91"/>
 <wire x1="129.54" y1="22.86" x2="132.08" y2="22.86" width="0.1524" layer="91"/>
-<wire x1="132.08" y1="22.86" x2="132.08" y2="35.56" width="0.1524" layer="91"/>
-<pinref part="SV2" gate="1" pin="5"/>
-<wire x1="152.4" y1="35.56" x2="132.08" y2="35.56" width="0.1524" layer="91"/>
+<wire x1="132.08" y1="22.86" x2="132.08" y2="38.1" width="0.1524" layer="91"/>
 <pinref part="IC2" gate="G$1" pin="OUTB"/>
 <junction x="129.54" y="22.86"/>
@@
 <junction x="129.54" y="15.24"/>
 <pinref part="IC2" gate="G$1" pin="OUTB@4"/>
+<pinref part="SV2" gate="1" pin="6"/>
+<wire x1="132.08" y1="38.1" x2="152.4" y2="38.1" width="0.1524" layer="91"/>
 </segment>
 </net>
@@
 <segment>
 <wire x1="129.54" y1="27.94" x2="129.54" y2="30.48" width="0.1524" layer="91"/>
-<pinref part="SV2" gate="1" pin="6"/>
 <wire x1="129.54" y1="30.48" x2="129.54" y2="33.02" width="0.1524" layer="91"/>
 <wire x1="129.54" y1="33.02" x2="129.54" y2="35.56" width="0.1524" layer="91"/>
 <wire x1="129.54" y1="35.56" x2="129.54" y2="38.1" width="0.1524" layer="91"/>
-<wire x1="129.54" y1="38.1" x2="152.4" y2="38.1" width="0.1524" layer="91"/>
 <pinref part="IC2" gate="G$1" pin="OUTA"/>
-<junction x="129.54" y="38.1"/>
 <pinref part="IC2" gate="G$1" pin="OUTA@1"/>
 <junction x="129.54" y="35.56"/>
@@
 <junction x="129.54" y="30.48"/>
 <pinref part="IC2" gate="G$1" pin="OUTA@4"/>
+<pinref part="SV2" gate="1" pin="5"/>
+<wire x1="152.4" y1="35.56" x2="129.54" y2="35.56" width="0.1524" layer="91"/>
 </segment>
 </net>
@@
 <net name="N$24" class="0">
 <segment>
-<wire x1="58.42" y1="35.56" x2="58.42" y2="25.4" width="0.1524" layer="91"/>
-<pinref part="U$1" gate="G$1" pin="PD5(XCK/CTS)"/>
-<wire x1="58.42" y1="25.4" x2="30.48" y2="25.4" width="0.1524" layer="91"/>
 <pinref part="R7" gate="G$1" pin="1"/>
-<pinref part="R15" gate="G$1" pin="2"/>
-<wire x1="88.9" y1="35.56" x2="58.42" y2="35.56" width="0.1524" layer="91"/>
+<wire x1="68.58" y1="96.52" x2="68.58" y2="35.56" width="0.1524" layer="91"/>
+<wire x1="68.58" y1="35.56" x2="58.42" y2="35.56" width="0.1524" layer="91"/>
+<wire x1="68.58" y1="96.52" x2="73.66" y2="96.52" width="0.1524" layer="91"/>
+<wire x1="73.66" y1="96.52" x2="76.2" y2="99.06" width="0.1524" layer="91"/>
+<pinref part="R12" gate="G$1" pin="2"/>
+<wire x1="76.2" y1="99.06" x2="88.9" y2="99.06" width="0.1524" layer="91"/>
+<wire x1="58.42" y1="35.56" x2="33.02" y2="35.56" width="0.1524" layer="91"/>
+<wire x1="33.02" y1="35.56" x2="33.02" y2="45.72" width="0.1524" layer="91"/>
 <junction x="58.42" y="35.56"/>
+<pinref part="U$1" gate="G$1" pin="PB4(ADC11)"/>
+<wire x1="33.02" y1="45.72" x2="30.48" y2="45.72" width="0.1524" layer="91"/>
 </segment>
 </net>
@@
 <pinref part="U$1" gate="G$1" pin="PD6(T1/ADC9/!OC4D)"/>
 <pinref part="R6" gate="G$1" pin="2"/>
-<pinref part="R13" gate="G$1" pin="2"/>
-<wire x1="88.9" y1="96.52" x2="58.42" y2="96.52" width="0.1524" layer="91"/>
+<pinref part="R15" gate="G$1" pin="2"/>
+<wire x1="88.9" y1="35.56" x2="86.36" y2="35.56" width="0.1524" layer="91"/>
+<wire x1="86.36" y1="35.56" x2="86.36" y2="86.36" width="0.1524" layer="91"/>
+<wire x1="86.36" y1="86.36" x2="66.04" y2="86.36" width="0.1524" layer="91"/>
+<wire x1="66.04" y1="86.36" x2="66.04" y2="96.52" width="0.1524" layer="91"/>
+<wire x1="66.04" y1="96.52" x2="58.42" y2="96.52" width="0.1524" layer="91"/>
 <junction x="58.42" y="96.52"/>
 </segment>
@@
 <pinref part="R9" gate="G$1" pin="2"/>
 <wire x1="63.5" y1="93.98" x2="63.5" y2="99.06" width="0.1524" layer="91"/>
-<pinref part="R12" gate="G$1" pin="2"/>
-<wire x1="88.9" y1="99.06" x2="63.5" y2="99.06" width="0.1524" layer="91"/>
+<pinref part="R13" gate="G$1" pin="2"/>
+<wire x1="88.9" y1="96.52" x2="76.2" y2="96.52" width="0.1524" layer="91"/>
+<wire x1="76.2" y1="96.52" x2="73.66" y2="99.06" width="0.1524" layer="91"/>
+<wire x1="73.66" y1="99.06" x2="63.5" y2="99.06" width="0.1524" layer="91"/>
 <junction x="63.5" y="99.06"/>
 </segment>

Commit message: finalizing layout
Parts:
- added S1: (no value), switch-omron:10-XX
Connections:
- removed net N$5: ISP1.RST, R1.2, U$1./RESET
- new net N$38: ISP1.RST, R1.2, S1.S, S1.S1, U$1./RESET
- net GND: now also S1.P, S1.P1
Changed lines of the file:
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@@
 <part name="IC1" library="st-microelectronics" deviceset="VNH3SP30" device=""/>
 <part name="IC2" library="st-microelectronics" deviceset="VNH3SP30" device=""/>
+<part name="S1" library="switch-omron" deviceset="10-XX" device=""/>
 </parts>
 <sheets>
@@
 <instance part="IC1" gate="G$1" x="114.3" y="88.9"/>
 <instance part="IC2" gate="G$1" x="114.3" y="25.4"/>
+<instance part="S1" gate="1" x="-40.64" y="88.9"/>
 </instances>
 <busses>
@@
 <wire x1="-53.34" y1="50.8" x2="-48.26" y2="50.8" width="0.1524" layer="91"/>
 <wire x1="-48.26" y1="50.8" x2="-48.26" y2="40.64" width="0.1524" layer="91"/>
-<wire x1="-48.26" y1="40.64" x2="-33.02" y2="40.64" width="0.1524" layer="91"/>
+<wire x1="-48.26" y1="40.64" x2="-40.64" y2="40.64" width="0.1524" layer="91"/>
+<pinref part="S1" gate="1" pin="P"/>
+<pinref part="S1" gate="1" pin="P1"/>
+<wire x1="-40.64" y1="40.64" x2="-33.02" y2="40.64" width="0.1524" layer="91"/>
+<wire x1="-40.64" y1="83.82" x2="-38.1" y2="83.82" width="0.1524" layer="91"/>
+<wire x1="-40.64" y1="83.82" x2="-40.64" y2="40.64" width="0.1524" layer="91"/>
+<junction x="-40.64" y="83.82"/>
+<junction x="-40.64" y="40.64"/>
 </segment>
 <segment>
@@
 </segment>
 </net>
-<net name="N$5" class="0">
-<segment>
-<pinref part="U$1" gate="G$1" pin="/RESET"/>
-<pinref part="R1" gate="G$1" pin="2"/>
-<wire x1="-17.78" y1="86.36" x2="-17.78" y2="93.98" width="0.1524" layer="91"/>
-<junction x="-17.78" y="86.36"/>
-<wire x1="-17.78" y1="93.98" x2="-2.54" y2="93.98" width="0.1524" layer="91"/>
-<wire x1="-2.54" y1="93.98" x2="-2.54" y2="101.6" width="0.1524" layer="91"/>
-<pinref part="ISP1" gate="G$1" pin="RST"/>
-<wire x1="-2.54" y1="101.6" x2="20.32" y2="101.6" width="0.1524" layer="91"/>
-</segment>
-</net>
 <net name="+12V" class="0">
 <segment>
@@
 </segment>
 </net>
+<net name="N$38" class="0">
+<segment>
+<pinref part="S1" gate="1" pin="S"/>
+<pinref part="S1" gate="1" pin="S1"/>
+<wire x1="-40.64" y1="93.98" x2="-38.1" y2="93.98" width="0.1524" layer="91"/>
+<pinref part="U$1" gate="G$1" pin="/RESET"/>
+<pinref part="R1" gate="G$1" pin="2"/>
+<wire x1="-17.78" y1="86.36" x2="-17.78" y2="93.98" width="0.1524" layer="91"/>
+<junction x="-17.78" y="86.36"/>
+<wire x1="-17.78" y1="93.98" x2="-2.54" y2="93.98" width="0.1524" layer="91"/>
+<wire x1="-2.54" y1="93.98" x2="-2.54" y2="101.6" width="0.1524" layer="91"/>
+<pinref part="ISP1" gate="G$1" pin="RST"/>
+<wire x1="-2.54" y1="101.6" x2="20.32" y2="101.6" width="0.1524" layer="91"/>
+<wire x1="-38.1" y1="93.98" x2="-17.78" y2="93.98" width="0.1524" layer="91"/>
+<junction x="-38.1" y="93.98"/>
+<junction x="-17.78" y="93.98"/>
+</segment>
+</net>

Commit message: finalizing layout
Parts:
- removed CN1: (no value), adafruit:USBMINIB
- removed IC1, IC2: VNH3SP30, st-microelectronics:VNH3SP30
- removed ISP1: AVRISP-6, adafruit:AVRISP-6
- removed Q1: (no value), adafruit:CRYSTALHC49U-V
- removed S1: (no value), switch-omron:10-XX
- removed SV1, SV2: (no value), con-lstb:MA06-1
- added C9: 2200u, rcl:CPOL-EUE5-8.5
- added J1: AVR_SPI_PRG_6NS, SparkFun-Connectors:AVR_SPI_PRG_6NS
- added JP1, JP2: (no value), SparkFun-Connectors:M06SIP
- added JP3: USB-SMD-NS, SparkFun-Connectors:USB-SMD-NS
- added S2: SWITCH-MOMENTARY-2PTH, SparkFun-Electromechanical:SWITCH-MOMENTARY-2PTH
- added U$2: ATMEGA32U4TQFP, SparkFun-DigitalIC:ATMEGA32U4TQFP
- added U$3: VNH2SP30, SparkFun-PowerIC:VNH2SP30
- added Y1: (no value), SparkFun-FreqCtrl:CRYSTALHC49US
- C1, C2, C3, C4, C5, C6, C7: device rcl:C-EUC0805K -> SparkFun-Passives:CAP0805
- LED1: value (none) -> A2; device led:LEDSML1206 -> SparkFun-LED:LED1206
- LED2: value (none) -> B1; device led:LEDSML1206 -> SparkFun-LED:LED1206
- LED3: value (none) -> A1; device led:LEDSML1206 -> SparkFun-LED:LED1206
- LED4: value (none) -> B2; device led:LEDSML1206 -> SparkFun-LED:LED1206
- LED5: value (none) -> +5V; device led:LEDSML1206 -> SparkFun-LED:LED1206
- LED6: value (none) -> +12V; device led:LEDSML1206 -> SparkFun-LED:LED1206
- R1: value (none) -> 10k; device rcl:R-EU_M0805 -> SparkFun-Passives:RESISTOR0805-RES
- R10, R11, R12, R13, R14, R15, R16, R17, R2, R3, R4, R5, R6, R7, R8, R9: device rcl:R-EU_M0805 -> SparkFun-Passives:RESISTOR0805-RES
- U$1: value ATMEGA32U4-AU -> VNH2SP30; device adafruit:ATMEGA32U4-AU -> SparkFun-PowerIC:VNH2SP30
Connections:
- removed net N$14: IC1.OUTB, IC1.OUTB@1, IC1.OUTB@2, IC1.OUTB@3, IC1.OUTB@4, SV1.5
- removed net N$15: IC2.OUTB, IC2.OUTB@1, IC2.OUTB@2, IC2.OUTB@3, IC2.OUTB@4, SV2.6
- removed net N$16: IC2.OUTA, IC2.OUTA@1, IC2.OUTA@2, IC2.OUTA@3, IC2.OUTA@4, SV2.5
- removed net N$18: IC2.DIAGA, R4.1
- removed net N$19: IC2.DIAGB, R5.1
- removed net N$21: IC1.DIAGB, R3.1
- removed net N$23: R16.2, R8.1, U$1.PD4(ICP1/ADC8)
- removed net N$24: R12.2, R7.1, U$1.PB4(ADC11)
- removed net N$25: R15.2, R6.2, U$1.PD6(T1/ADC9/!OC4D)
- removed net N$26: R13.2, R9.2, U$1.PD7(OC4D/ADC10/T0)
- removed net N$32: IC1.INA, R12.1
- removed net N$33: IC1.INB, R13.1
- removed net N$34: IC1.PWM, R14.1
- removed net N$35: IC2.INA, R15.1
- removed net N$36: IC2.INB, R16.1
- removed net N$37: IC2.PWM, R17.1
- new net N$5: R16.1, U$1.INB
- new net OUTA1: JP1.1, U$3.OUTA@1, U$3.OUTA@25, U$3.OUTA@30, U$3.OUTA@SLUG3
- new net OUTA2: JP2.2, U$1.OUTA@1, U$1.OUTA@25, U$1.OUTA@30, U$1.OUTA@SLUG3
- new net OUTB1: JP1.2, U$3.OUTB@15, U$3.OUTB@16, U$3.OUTB@21, U$3.OUTB@SLUG2
- new net OUTB2: JP2.1, U$1.OUTB@15, U$1.OUTB@16, U$1.OUTB@21, U$1.OUTB@SLUG2
- new net PB0: U$2.PB0(SS)
- new net PB1: J1.3, U$2.PB1(SCK)
- new net PB2: J1.4, U$2.PB2(MOSI)
- new net PB3: J1.1, U$2.PB3(MISO)
- new net PB4: R12.2, R7.1, U$2.PB4(ADC11)
- new net PB5: R17.2, U$2.PB5(ADC12)
- new net PB6: R14.2, U$2.PB6(ADC13)
- new net PB7: U$2.PB7
- new net PC6: U$2.PC6
- new net PC7: U$2.PC7
- new net PD0: JP2.6, U$2.PD0(SCL)
- new net PD1: JP1.6, U$2.PD1(SDA)
- new net PD2: U$2.PD2(RX)
- new net PD3: U$2.PD3(TX)
- new net PD4: R16.2, R8.1, U$2.PD4(ADC8)
- new net PD5: U$2.PD5
- new net PD6: R15.2, R6.2, U$2.PD6(ADC9)
- new net PD7: R13.2, R9.2, U$2.PD7(ADC10)
- new net PE6: U$2.PE6
- net +12V: now also C9.+, U$1.VCC@13, U$1.VCC@23, U$1.VCC@3, U$1.VCC@SLUG1, U$3.VCC@13, U$3.VCC@23, U$3.VCC@3, U$3.VCC@SLUG1; no longer IC1.VCC, IC1.VCC@1, IC1.VCC@2, IC1.VCC@3, IC1.VCC@4, IC2.VCC, IC2.VCC@1, IC2.VCC@2, IC2.VCC@3, IC2.VCC@4
- net +5V: now also J1.2, JP1.4, JP2.4, JP3.VBUS, U$2.AVCC@24, U$2.AVCC@44, U$2.UVCC, U$2.VBUS, U$2.VCC@14, U$2.VCC@34; no longer CN1.VBUS, ISP1.VCC, SV1.3, SV2.3, U$1.AVCC, U$1.AVCC1, U$1.UVCC, U$1.VBUS, U$1.VCC, U$1.VCC1
- net GND: now also C9.-, J1.6, JP1.3, JP2.3, JP3.GND, S2.1, U$1.GNDA@26, U$1.GNDA@27, U$1.GNDA@28, U$1.GNDB@18, U$1.GNDB@19, U$1.GNDB@20, U$2.GND@15, U$2.GND@23, U$2.GND@35, U$2.GND@43, U$2.UGND, U$3.GNDA@26, U$3.GNDA@27, U$3.GNDA@28, U$3.GNDB@18, U$3.GNDB@19, U$3.GNDB@20; no longer CN1.GND, IC1.GNDA, IC1.GNDA@1, IC1.GNDA@2, IC1.GNDB, IC1.GNDB@1, IC1.GNDB@2, IC2.GNDA, IC2.GNDA@1, IC2.GNDA@2, IC2.GNDB, IC2.GNDB@1, IC2.GNDB@2, ISP1.GND, S1.P, S1.P1, SV1.4, SV2.4, U$1.GND, U$1.GND1, U$1.GND2, U$1.GND3, U$1.UGND
- net N$1: now also R15.1, U$1.INA; no longer ISP1.SCK, U$1.PB1(SCK)
- net N$10: now also JP3.D+, U$2.D+; no longer CN1.D+, U$1.D+
- net N$11: now also JP3.D-, U$2.D-; no longer CN1.D-, U$1.D-
- net N$12: now also R13.1, U$3.INB; no longer SV2.1, U$1.PD0(INT0/OC0B/SCL)
- net N$13: now also R14.1, U$3.PWM; no longer IC1.OUTA, IC1.OUTA@1, IC1.OUTA@2, IC1.OUTA@3, IC1.OUTA@4, SV1.6
- net N$17: now also R3.1, U$3.EN/DIAB; no longer SV1.1, U$1.PD1(INT1/SDA)
- net N$2: now also U$2.XTAL2, Y1.1; no longer Q1.1, U$1.XTAL2
- net N$20: now also U$3.EN/DIAA; no longer IC1.DIAGA
- net N$3: now also U$2.XTAL1, Y1.2; no longer Q1.2, U$1.XTAL1
- net N$38: now also J1.5, S2.2, U$2.!RESET; no longer ISP1.RST, S1.S, S1.S1, U$1./RESET
- net N$4: now also U$2.UCAP; no longer U$1.UCAP
- net N$6: now also R17.1, U$1.PWM; no longer ISP1.MOSI, U$1.PB2(PDI/MOSI)
- net N$7: now also R5.1, U$1.EN/DIAB; no longer ISP1.MISO, U$1.PB3(PDO/MISO)
- net N$8: now also R4.1, U$1.EN/DIAA; no longer R17.2, U$1.PB5(OC1A/ADC12/!OC4B)
- net N$9: now also R12.1, U$3.INA; no longer R14.2, U$1.PB6(OC1B/OC4B/ADC13)
Other:
- moved on the sheet: C3
